File: Hardware/Diseño PCB/Buck/Buck.kicad_pcb (KiCad board)
At the start: 2 copper layers, 28 parts, among them Q1 NMOS, Q2 NMOS, Q3 BC546, U1 TL431D, U2 IR2111, U3 TL082, U4 TL082

Commit message: CHK4: Informe + pcb
Parts:
- removed U1: TL431D, Package_SO:SOIC-8_3.9x4.9mm_P1.27mm
- added U5: TL431LP, Package_TO_SOT_THT:TO-92_HandSolder, F.Cu at (172.0, 83.0)
- Q3: footprint Package_TO_SOT_THT:TO-92_Inline -> Package_TO_SOT_THT:TO-92_HandSolder
- moved U3 86.7 mm to (115.1, 82.0)
- moved D1 85.9 mm to (190.5, 65.5)
- moved U4 84.2 mm to (135.5, 82.0)
- moved C3 73.4 mm to (110.4, 93.5)
- moved R11 69.7 mm to (185.2, 90.8), turned to 180 degrees
- moved R10 68.5 mm to (133.6, 64.9), turned to 180 degrees
- moved C4 67.2 mm to (120.1, 93.4)
- moved R3 66.9 mm to (181.7, 66.0), turned to -90 degrees
- moved Vo1 65.1 mm to (193.0, 54.0)
- moved VEE1 64.9 mm to (106.0, 49.0)
- moved R4 64.6 mm to (175.2, 66.0), turned to -90 degrees
- moved R12 63.8 mm to (173.5, 90.8), turned to 180 degrees
- moved Q2 62.5 mm to (102.4, 87.5), turned to 90 degrees
- moved U2 58.0 mm to (110.4, 107.1), turned to 90 degrees
- moved R5 57.0 mm to (168.7, 73.6), turned to 90 degrees
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Other:
- board outline added: 106.5 x 67.5 mm
