File: Hardware/Diseño PCB/PWM/pwm.kicad_pcb (KiCad board)
At the start: 2 copper layers, 100 x 80 mm, 38 parts, among them J1 VE, J2 Vo, Q3 IRF540N, Q4 IRF540N, U2 IR2111

Commit message: CHK4: Correccion pcb NMOS
Parts:
- added BC546: BC546, Package_TO_SOT_THT:TO-92_HandSolder, F.Cu at (39.0, 259.1)
- added BC546: BC546, Package_TO_SOT_THT:TO-92_HandSolder, F.Cu at (39.1, 175.6)
- added C1: 100u, Capacitor_THT:CP_Radial_D10.0mm_P2.50mm, F.Cu at (43.2, 205.6)
- added C1: 100u, Capacitor_THT:CP_Radial_D10.0mm_P2.50mm, F.Cu at (43.3, 122.1)
- added C2: 100u, Capacitor_THT:CP_Radial_D10.0mm_P2.50mm, F.Cu at (97.5, 205.6)
- added C2: 100u, Capacitor_THT:CP_Radial_D10.0mm_P2.50mm, F.Cu at (97.6, 122.1)
- added C3: 10u, Capacitor_THT:C_Disc_D6.0mm_W4.4mm_P5.00mm, F.Cu at (65.7, 239.8)
- added C3: 10u, Capacitor_THT:C_Disc_D6.0mm_W4.4mm_P5.00mm, F.Cu at (65.8, 156.2)
- added C4: 1n, Capacitor_THT:C_Disc_D6.0mm_W4.4mm_P5.00mm, F.Cu at (75.3, 257.8)
- added C4: 1n, Capacitor_THT:C_Disc_D6.0mm_W4.4mm_P5.00mm, F.Cu at (75.4, 174.2)
- added C5: 10n, Capacitor_THT:C_Disc_D6.0mm_W4.4mm_P5.00mm, F.Cu at (89.3, 225.7)
- added C5: 10n, Capacitor_THT:C_Disc_D6.0mm_W4.4mm_P5.00mm, F.Cu at (89.4, 142.1)
- added C6: 1n, Capacitor_THT:C_Disc_D6.0mm_W4.4mm_P5.00mm, F.Cu at (99.4, 225.8)
- added C6: 1n, Capacitor_THT:C_Disc_D6.0mm_W4.4mm_P5.00mm, F.Cu at (99.5, 142.2)
- added D1: LED, LED_THT:LED_D4.0mm, F.Cu at (114.7, 195.2)
- added D1: LED, LED_THT:LED_D4.0mm, F.Cu at (114.8, 111.7)
- added GND1: GND, Connector_PinHeader_2.00mm:PinHeader_1x01_P2.00mm_Vertical, F.Cu at (28.3, 147.0)
- added GND1: GND, Connector_PinHeader_2.00mm:PinHeader_1x01_P2.00mm_Vertical, F.Cu at (28.2, 230.6)
- added J1: VE, TerminalBlock_Phoenix:TerminalBlock_Phoenix_MKDS-1,5-2_1x02_P5.00mm_Horizontal, F.Cu at (31.5, 121.1)
- added J1: VE, TerminalBlock_Phoenix:TerminalBlock_Phoenix_MKDS-1,5-2_1x02_P5.00mm_Horizontal, F.Cu at (31.4, 204.7)
- added J2: Vo, TerminalBlock_Phoenix:TerminalBlock_Phoenix_MKDS-1,5-2_1x02_P5.00mm_Horizontal, F.Cu at (115.8, 126.3)
- added J2: Vo, TerminalBlock_Phoenix:TerminalBlock_Phoenix_MKDS-1,5-2_1x02_P5.00mm_Horizontal, F.Cu at (115.7, 209.8)
- added L1: 50u, Inductor_THT:L_Axial_L20.0mm_D8.0mm_P25.40mm_Horizontal, F.Cu at (59.2, 205.7)
- added L1: 50u, Inductor_THT:L_Axial_L20.0mm_D8.0mm_P25.40mm_Horizontal, F.Cu at (59.3, 122.2)
- added LM319: LM319, Package_DIP:DIP-8_W7.62mm_Socket, F.Cu at (95.6, 241.8)
- added LM319: LM319, Package_DIP:DIP-8_W7.62mm_Socket, F.Cu at (95.7, 158.2)
- added MBR735: MBR735, Package_TO_SOT_THT:TO-220-2_Vertical, F.Cu at (62.1, 261.2)
- added MBR735: MBR735, Package_TO_SOT_THT:TO-220-2_Vertical, F.Cu at (62.2, 177.6)
- added Q3: IRF540N, Package_TO_SOT_THT:TO-220-3_Vertical, F.Cu at (60.7, 194.0)
- added Q3: IRF540N, Package_TO_SOT_THT:TO-220-3_Vertical, F.Cu at (60.8, 110.4)
- added Q4: IRF540N, Package_TO_SOT_THT:TO-220-3_Vertical, F.Cu at (78.3, 110.4)
- added Q4: IRF540N, Package_TO_SOT_THT:TO-220-3_Vertical, F.Cu at (78.2, 194.0)
- added R1: 10k, Resistor_THT:R_Axial_DIN0204_L3.6mm_D1.6mm_P7.62mm_Horizontal, F.Cu at (116.5, 147.6)
- added R1: 10k, Resistor_THT:R_Axial_DIN0204_L3.6mm_D1.6mm_P7.62mm_Horizontal, F.Cu at (116.4, 231.2)
- added R10: 10k, Resistor_THT:R_Axial_DIN0204_L3.6mm_D1.6mm_P7.62mm_Horizontal, F.Cu at (84.3, 150.9)
- added R10: 10k, Resistor_THT:R_Axial_DIN0204_L3.6mm_D1.6mm_P7.62mm_Horizontal, F.Cu at (84.2, 234.5)
- added R11: 100k, Resistor_THT:R_Axial_DIN0204_L3.6mm_D1.6mm_P7.62mm_Horizontal, F.Cu at (44.4, 158.4)
- added R11: 100k, Resistor_THT:R_Axial_DIN0204_L3.6mm_D1.6mm_P7.62mm_Horizontal, F.Cu at (44.3, 242.0)
- added R12: 100k, Resistor_THT:R_Axial_DIN0204_L3.6mm_D1.6mm_P7.62mm_Horizontal, F.Cu at (44.4, 252.7)
- added R12: 100k, Resistor_THT:R_Axial_DIN0204_L3.6mm_D1.6mm_P7.62mm_Horizontal, F.Cu at (44.5, 169.1)
- added R13: 100, Resistor_THT:R_Axial_DIN0204_L3.6mm_D1.6mm_P7.62mm_Horizontal, F.Cu at (113.1, 179.0)
- added R13: 100, Resistor_THT:R_Axial_DIN0204_L3.6mm_D1.6mm_P7.62mm_Horizontal, F.Cu at (113.0, 262.5)
- added R14: 1k, Resistor_THT:R_Axial_DIN0204_L3.6mm_D1.6mm_P7.62mm_Horizontal, F.Cu at (80.7, 146.0)
- added R14: 1k, Resistor_THT:R_Axial_DIN0204_L3.6mm_D1.6mm_P7.62mm_Horizontal, F.Cu at (80.6, 229.6)
- added R15: 30k, Resistor_THT:R_Axial_DIN0204_L3.6mm_D1.6mm_P7.62mm_Horizontal, F.Cu at (72.8, 151.0)
- added R15: 30k, Resistor_THT:R_Axial_DIN0204_L3.6mm_D1.6mm_P7.62mm_Horizontal, F.Cu at (72.7, 234.6)
- added R2: 10k, Resistor_THT:R_Axial_DIN0204_L3.6mm_D1.6mm_P7.62mm_Horizontal, F.Cu at (116.5, 160.4)
- added R2: 10k, Resistor_THT:R_Axial_DIN0204_L3.6mm_D1.6mm_P7.62mm_Horizontal, F.Cu at (116.4, 244.0)
- added R3: 1k, Resistor_THT:R_Axial_DIN0204_L3.6mm_D1.6mm_P7.62mm_Horizontal, F.Cu at (35.5, 167.4)
- added R3: 1k, Resistor_THT:R_Axial_DIN0204_L3.6mm_D1.6mm_P7.62mm_Horizontal, F.Cu at (35.4, 251.0)
- added R4: 1k, Resistor_THT:R_Axial_DIN0204_L3.6mm_D1.6mm_P7.62mm_Horizontal, F.Cu at (35.5, 160.9)
- added R4: 1k, Resistor_THT:R_Axial_DIN0204_L3.6mm_D1.6mm_P7.62mm_Horizontal, F.Cu at (35.4, 244.5)
- added R5: 1k, Resistor_THT:R_Axial_DIN0204_L3.6mm_D1.6mm_P7.62mm_Horizontal, F.Cu at (35.5, 154.9)
- added R5: 1k, Resistor_THT:R_Axial_DIN0204_L3.6mm_D1.6mm_P7.62mm_Horizontal, F.Cu at (35.4, 238.5)
- added R6: 33k, Resistor_THT:R_Axial_DIN0204_L3.6mm_D1.6mm_P7.62mm_Horizontal, F.Cu at (81.5, 179.0)
- added R6: 33k, Resistor_THT:R_Axial_DIN0204_L3.6mm_D1.6mm_P7.62mm_Horizontal, F.Cu at (81.3, 262.5)
- added R7: 100k, Resistor_THT:R_Axial_DIN0204_L3.6mm_D1.6mm_P7.62mm_Horizontal, F.Cu at (92.1, 179.0)
- added R7: 100k, Resistor_THT:R_Axial_DIN0204_L3.6mm_D1.6mm_P7.62mm_Horizontal, F.Cu at (92.0, 262.5)
- added R8: 5k6, Resistor_THT:R_Axial_DIN0204_L3.6mm_D1.6mm_P7.62mm_Horizontal, F.Cu at (102.6, 179.0)
- added R8: 5k6, Resistor_THT:R_Axial_DIN0204_L3.6mm_D1.6mm_P7.62mm_Horizontal, F.Cu at (102.5, 262.5)
- added R9: 22k, Resistor_THT:R_Axial_DIN0204_L3.6mm_D1.6mm_P7.62mm_Horizontal, F.Cu at (106.3, 234.5)
- added R9: 22k, Resistor_THT:R_Axial_DIN0204_L3.6mm_D1.6mm_P7.62mm_Horizontal, F.Cu at (106.4, 150.9)
- added TL082: TL082, Package_DIP:DIP-8_W7.62mm_Socket, F.Cu at (75.9, 158.2)
- added TL082: TL082, Package_DIP:DIP-8_W7.62mm_Socket, F.Cu at (75.8, 241.8)
- added TL431: TL431LP, Package_TO_SOT_THT:TO-92_HandSolder, F.Cu at (30.5, 258.9)
- added TL431: TL431LP, Package_TO_SOT_THT:TO-92_HandSolder, F.Cu at (30.6, 175.3)
- added U2: IR2111, Package_DIP:DIP-8_W7.62mm_Socket, F.Cu at (53.4, 247.0)
- added U2: IR2111, Package_DIP:DIP-8_W7.62mm_Socket, F.Cu at (53.5, 163.4)
- added VEE1: VEE, Connector_PinHeader_2.00mm:PinHeader_1x01_P2.00mm_Vertical, F.Cu at (28.2, 225.5)
- added VEE1: VEE, Connector_PinHeader_2.00mm:PinHeader_1x01_P2.00mm_Vertical, F.Cu at (28.3, 141.9)
- added Vctrl_H1: Vctrl_H, Connector_PinHeader_2.00mm:PinHeader_1x01_P2.00mm_Vertical, F.Cu at (54.7, 223.4)
- added Vctrl_H1: Vctrl_H, Connector_PinHeader_2.00mm:PinHeader_1x01_P2.00mm_Vertical, F.Cu at (54.8, 139.9)
- added Vctrl_L1: Vctrl_L, Connector_PinHeader_2.00mm:PinHeader_1x01_P2.00mm_Vertical, F.Cu at (63.0, 223.4)
- added Vctrl_L1: Vctrl_L, Connector_PinHeader_2.00mm:PinHeader_1x01_P2.00mm_Vertical, F.Cu at (63.1, 139.9)
- added Vo1: Vo, Connector_PinHeader_2.00mm:PinHeader_1x01_P2.00mm_Vertical, F.Cu at (116.5, 142.2)
- added Vo1: Vo, Connector_PinHeader_2.00mm:PinHeader_1x01_P2.00mm_Vertical, F.Cu at (116.3, 225.7)
- moved C1 70.9 mm to (43.2, 35.4)
- moved C3 70.9 mm to (65.7, 69.5)
- moved C4 70.9 mm to (75.2, 87.5)
- moved C5 70.9 mm to (89.2, 55.4)
- moved C6 70.9 mm to (99.3, 55.5)
- moved D1 70.9 mm to (114.6, 25.0)
- moved J1 70.9 mm to (31.3, 34.4)
- moved L1 70.9 mm to (59.1, 35.4)
- moved MBR735 70.9 mm to (62.1, 90.9)
- moved Q3 70.9 mm to (60.6, 23.7)
- moved R12 70.9 mm to (44.4, 82.4)
- moved R3 70.9 mm to (35.4, 80.7)
- moved R4 70.9 mm to (35.4, 74.2)
- moved R5 70.9 mm to (35.4, 68.2)
- moved VEE1 70.9 mm to (28.1, 55.2)
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- renumbered D2 to MBR735
Routing:
- net /VEE: track 225.6 -> 676.8 mm
- net /PWM: track 172.0 -> 515.9 mm
- net GND: track 156.9 -> 470.6 mm
- net /Vcc5: track 131.3 -> 393.9 mm
- net /Vo: track 113.7 -> 341.0 mm
- net /Vctrl_L: track 105.8 -> 317.3 mm
- net /Vmed: track 93.0 -> 279.0 mm
- net /Vctrl_H: track 83.7 -> 251.1 mm
- net Net-(TL082B--): track 64.8 -> 194.4 mm
- net /v_muestra: track 53.4 -> 160.1 mm
- net Net-(TL082A--): track 51.5 -> 154.5 mm
- net Net-(Q3-S): track 34.3 -> 103.0 mm
- net Net-(LM319B-+): track 33.9 -> 101.6 mm
- net Net-(BC546-B): track 30.5 -> 91.6 mm
- net Net-(D2-K): track 29.0 -> 86.9 mm
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Other:
- board size 100 x 80 mm -> 100.2 x 250.3 mm

Commit message: CHK4: Informe
Parts:
- removed the BC546 at (39.0, 259.1)
- removed the BC546 at (39.1, 175.6)
- removed the C1 at (43.2, 205.6)
- removed the C1 at (43.3, 122.1)
- removed the C2 at (97.5, 205.6)
- removed the C2 at (97.6, 122.1)
- removed the C3 at (65.7, 239.8)
- removed the C3 at (65.8, 156.2)
- removed the C4 at (75.3, 257.8)
- removed the C4 at (75.4, 174.2)
- removed the C5 at (89.3, 225.7)
- removed the C5 at (89.4, 142.1)
- removed the C6 at (99.4, 225.8)
- removed the C6 at (99.5, 142.2)
- removed the D1 at (114.7, 195.2)
- removed the D1 at (114.8, 111.7)
- removed the GND1 at (28.3, 147.0)
- removed the GND1 at (28.2, 230.6)
- removed the J1 at (31.5, 121.1)
- removed the J1 at (31.4, 204.7)
- removed the J2 at (115.8, 126.3)
- removed the J2 at (115.7, 209.8)
- removed the L1 at (59.2, 205.7)
- removed the L1 at (59.3, 122.2)
- removed the LM319 at (95.6, 241.8)
- removed the LM319 at (95.7, 158.2)
- removed the MBR735 at (62.1, 261.2)
- removed the MBR735 at (62.2, 177.6)
- removed the Q3 at (60.7, 194.0)
- removed the Q3 at (60.8, 110.4)
- removed the Q4 at (78.3, 110.4)
- removed the Q4 at (78.2, 194.0)
- removed the R1 at (116.5, 147.6)
- removed the R1 at (116.4, 231.2)
- removed the R10 at (84.3, 150.9)
- removed the R10 at (84.2, 234.5)
- removed the R11 at (44.4, 158.4)
- removed the R11 at (44.3, 242.0)
- removed the R12 at (44.4, 252.7)
- removed the R12 at (44.5, 169.1)
- removed the R13 at (113.1, 179.0)
- removed the R13 at (113.0, 262.5)
- removed the R14 at (80.7, 146.0)
- removed the R14 at (80.6, 229.6)
- removed the R15 at (72.8, 151.0)
- removed the R15 at (72.7, 234.6)
- removed the R2 at (116.5, 160.4)
- removed the R2 at (116.4, 244.0)
- removed the R3 at (35.5, 167.4)
- removed the R3 at (35.4, 251.0)
- removed the R4 at (35.5, 160.9)
- removed the R4 at (35.4, 244.5)
- removed the R5 at (35.5, 154.9)
- removed the R5 at (35.4, 238.5)
- removed the R6 at (81.5, 179.0)
- removed the R6 at (81.3, 262.5)
- removed the R7 at (92.1, 179.0)
- removed the R7 at (92.0, 262.5)
- removed the R8 at (102.6, 179.0)
- removed the R8 at (102.5, 262.5)
- removed the R9 at (106.3, 234.5)
- removed the R9 at (106.4, 150.9)
- removed the TL082 at (75.9, 158.2)
- removed the TL082 at (75.8, 241.8)
- removed the TL431 at (30.5, 258.9)
- removed the TL431 at (30.6, 175.3)
- removed the U2 at (53.4, 247.0)
- removed the U2 at (53.5, 163.4)
- removed the VEE1 at (28.2, 225.5)
- removed the VEE1 at (28.3, 141.9)
- removed the Vctrl_H1 at (54.7, 223.4)
- removed the Vctrl_H1 at (54.8, 139.9)
- removed the Vctrl_L1 at (63.0, 223.4)
- removed the Vctrl_L1 at (63.1, 139.9)
- removed the Vo1 at (116.5, 142.2)
- removed the Vo1 at (116.3, 225.7)
- moved C6 30.8 mm to (129.8, 60.2)
- moved D1 30.8 mm to (145.1, 29.7)
- moved R7 30.8 mm to (122.4, 97.0)
- moved Vo1 30.8 mm to (146.7, 60.2)
- moved C1 30.8 mm to (73.6, 40.1)
- moved GND1 30.8 mm to (58.6, 65.0)
- moved L1 30.8 mm to (89.6, 40.2)
- moved MBR735 30.8 mm to (92.5, 95.7)
- moved Q3 30.8 mm to (91.0, 28.5)
- moved R12 30.8 mm to (74.8, 87.2)
- moved R3 30.8 mm to (65.8, 85.5)
- moved R4 30.8 mm to (65.8, 79.0)
- moved R5 30.8 mm to (65.8, 73.0)
- moved VEE1 30.8 mm to (58.6, 60.0)
- moved Vctrl_H1 30.8 mm to (85.1, 57.9)
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Routing:
- net /VEE: track 676.8 -> 229.7 mm
- net /PWM: track 515.9 -> 172.0 mm
- net GND: track 470.6 -> 156.9 mm
- net /Vctrl_L: track 317.3 -> 40.1 mm
- net /Vcc5: track 393.9 -> 131.3 mm
- net /Vo: track 341.0 -> 109.6 mm
- net /Vmed: track 279.0 -> 93.0 mm
- net /Vctrl_H: track 251.1 -> 83.7 mm
- net /v_muestra: track 160.1 -> 53.4 mm
- net Net-(TL082A--): track 154.5 -> 51.5 mm
- net Net-(TL082B--): track 194.4 -> 93.8 mm
- net Net-(D2-K): track 86.9 -> 0.00 mm
- net Net-(LM319B-+): track 101.6 -> 33.9 mm
- net Net-(BC546-B): track 91.6 -> 30.5 mm
- net /V_triag: track 82.9 -> 27.6 mm
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Other:
- board size 100.2 x 250.3 mm -> 100 x 80 mm

Commit message: CHK4: Informe
Parts:
- moved MBR735 6.86 mm to (89.1, 89.7)
- moved R7 6.86 mm to (119.0, 91.0)
- moved GND1 6.86 mm to (55.2, 59.1)
- moved C1 6.86 mm to (70.2, 34.2)
- moved C3 6.86 mm to (92.7, 68.3)
- moved C6 6.86 mm to (126.4, 54.3)
- moved D1 6.86 mm to (141.7, 23.8)
- moved R14 6.86 mm to (107.6, 58.1)
- moved R6 6.86 mm to (108.3, 91.0)
- moved R9 6.86 mm to (133.3, 63.0)
- moved Vo1 6.86 mm to (143.3, 54.3)
- moved VEE1 6.86 mm to (55.2, 54.0)
- moved C2 6.86 mm to (124.5, 34.2)
- moved L1 6.86 mm to (86.2, 34.2)
- moved Q3 6.86 mm to (87.7, 22.5)
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Routing:
- net /VEE: track 229.7 -> 451.2 mm
- net /PWM: track 172.0 -> 344.0 mm
- net /Vctrl_L: track 40.1 -> 211.5 mm
- net GND: track 156.9 -> 313.7 mm
- net /Vcc5: track 131.3 -> 262.6 mm
- net /Vo: track 109.6 -> 227.3 mm
- net /Vmed: track 93.0 -> 186.0 mm
- net /Vctrl_H: track 83.7 -> 167.4 mm
- net Net-(D2-K): track 0.00 -> 57.9 mm
- net /v_muestra: track 53.4 -> 106.7 mm
- net Net-(TL082A--): track 51.5 -> 103.0 mm
- net Net-(TL082B--): track 93.8 -> 129.6 mm
- net Net-(LM319B-+): track 33.9 -> 67.7 mm
- net Net-(Q3-S): track 100.0 -> 68.7 mm
- net Net-(BC546-B): track 30.5 -> 61.0 mm
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Other:
- board size 100 x 80 mm -> 100.3 x 249.4 mm

Commit message: Placa BuckV1
Parts:
- removed LM319: LM319, Package_DIP:DIP-8_W7.62mm_Socket
- removed TL082: TL082, Package_DIP:DIP-8_W7.62mm_Socket
- removed the U2 at (80.4, 75.5)
- added ?: , , F.Cu at (53.4, 105.1)
- added ?: , , F.Cu at (70.9, 177.9)
- added ?: , , F.Cu at (144.8, 86.0)
- added ?: , , F.Cu at (53.4, 194.1)
- added ?: , , F.Cu at (70.9, 266.9)
- added ?: , , F.Cu at (144.1, 260.1)
- added ?: , , F.Cu at (71.5, 92.8)
- added ?: , , F.Cu at (54.0, 20.0)
- added ?: , , F.Cu at (144.1, 171.1)
- added BC1: ~, Package_TO_SOT_THT:TO-92_HandSolder, F.Cu at (65.3, 261.8)
- added BC1: ~, Package_TO_SOT_THT:TO-92_HandSolder, F.Cu at (65.3, 172.8)
- added C1: 100u, Capacitor_THT:CP_Radial_D10.0mm_P2.50mm, F.Cu at (69.6, 208.3)
- added C1: 100u, Capacitor_THT:CP_Radial_D10.0mm_P2.50mm, F.Cu at (69.6, 119.3)
- added C2: 1n, Capacitor_THT:C_Disc_D6.0mm_W4.4mm_P5.00mm, F.Cu at (125.7, 139.4)
- added C2: 1n, Capacitor_THT:C_Disc_D6.0mm_W4.4mm_P5.00mm, F.Cu at (125.7, 228.4)
- added C3: 100u, Capacitor_THT:CP_Radial_D10.0mm_P2.50mm, F.Cu at (123.8, 208.3)
- added C3: 100u, Capacitor_THT:CP_Radial_D10.0mm_P2.50mm, F.Cu at (123.8, 119.3)
- added C4: 10n, Capacitor_THT:C_Disc_D6.0mm_W4.4mm_P5.00mm, F.Cu at (115.6, 228.3)
- added C4: 10n, Capacitor_THT:C_Disc_D6.0mm_W4.4mm_P5.00mm, F.Cu at (115.6, 139.3)
- added C5: 1n, Capacitor_THT:C_Disc_D6.0mm_W4.4mm_P5.00mm, F.Cu at (101.6, 260.4)
- added C5: 1n, Capacitor_THT:C_Disc_D6.0mm_W4.4mm_P5.00mm, F.Cu at (101.6, 171.4)
- added C6: 10u, Capacitor_THT:C_Disc_D6.0mm_W4.4mm_P5.00mm, F.Cu at (92.1, 242.4)
- added C6: 10u, Capacitor_THT:C_Disc_D6.0mm_W4.4mm_P5.00mm, F.Cu at (92.1, 153.4)
- added D1: LED, LED_THT:LED_D4.0mm, F.Cu at (141.0, 108.9)
- added D1: LED, LED_THT:LED_D4.0mm, F.Cu at (141.0, 197.9)
- added D2: MBR735, Package_TO_SOT_THT:TO-220-2_Vertical, F.Cu at (88.5, 263.8)
- added D2: MBR735, Package_TO_SOT_THT:TO-220-2_Vertical, F.Cu at (88.5, 174.8)
- added GND1: GND, Connector_PinHeader_2.00mm:PinHeader_1x01_P2.00mm_Vertical, F.Cu at (54.5, 233.2)
- added GND1: GND, Connector_PinHeader_2.00mm:PinHeader_1x01_P2.00mm_Vertical, F.Cu at (54.5, 144.2)
- added J1: VE, TerminalBlock_Phoenix:TerminalBlock_Phoenix_MKDS-1,5-2_1x02_P5.00mm_Horizontal, F.Cu at (57.7, 207.3)
- added J1: VE, TerminalBlock_Phoenix:TerminalBlock_Phoenix_MKDS-1,5-2_1x02_P5.00mm_Horizontal, F.Cu at (57.7, 118.3)
- added J2: V_triag, Connector_PinHeader_2.00mm:PinHeader_1x01_P2.00mm_Vertical, F.Cu at (108.5, 87.0)
- added J2: V_triag, Connector_PinHeader_2.00mm:PinHeader_1x01_P2.00mm_Vertical, F.Cu at (107.9, 261.1)
- added J2: V_triag, Connector_PinHeader_2.00mm:PinHeader_1x01_P2.00mm_Vertical, F.Cu at (107.9, 172.1)
- added J3: sense, Connector_PinHeader_2.00mm:PinHeader_1x02_P2.00mm_Vertical, F.Cu at (140.9, 158.6)
- added J3: sense, Connector_PinHeader_2.00mm:PinHeader_1x02_P2.00mm_Vertical, F.Cu at (141.5, 73.5)
- added J3: sense, Connector_PinHeader_2.00mm:PinHeader_1x02_P2.00mm_Vertical, F.Cu at (140.9, 247.6)
- added J4: Vo, TerminalBlock_Phoenix:TerminalBlock_Phoenix_MKDS-1,5-2_1x02_P5.00mm_Horizontal, F.Cu at (142.1, 123.5)
- added J4: Vo, TerminalBlock_Phoenix:TerminalBlock_Phoenix_MKDS-1,5-2_1x02_P5.00mm_Horizontal, F.Cu at (142.1, 212.5)
- added J5: pwm, Connector_PinHeader_2.00mm:PinHeader_1x02_P2.00mm_Vertical, F.Cu at (111.8, 58.0)
- added J5: pwm, Connector_PinHeader_2.00mm:PinHeader_1x02_P2.00mm_Vertical, F.Cu at (111.1, 232.1)
- added J5: pwm, Connector_PinHeader_2.00mm:PinHeader_1x02_P2.00mm_Vertical, F.Cu at (111.1, 143.1)
- added L1: 50u, Inductor_THT:L_Axial_L20.0mm_D8.0mm_P25.40mm_Horizontal, F.Cu at (85.5, 208.3)
- added L1: 50u, Inductor_THT:L_Axial_L20.0mm_D8.0mm_P25.40mm_Horizontal, F.Cu at (85.5, 119.3)
- added LM1: LM319, Package_DIP:DIP-14_W7.62mm_Socket, F.Cu at (119.2, 252.9)
- added LM1: LM319, Package_DIP:DIP-14_W7.62mm_Socket, F.Cu at (119.2, 163.9)
- added LM1: LM319, Package_DIP:DIP-14_W7.62mm_Socket, F.Cu at (119.8, 78.8)
- added Q1: IRF540N, Package_TO_SOT_THT:TO-220-3_Vertical, F.Cu at (87.0, 107.6)
- added Q1: IRF540N, Package_TO_SOT_THT:TO-220-3_Vertical, F.Cu at (87.0, 196.6)
- added Q2: IRF540N, Package_TO_SOT_THT:TO-220-3_Vertical, F.Cu at (104.5, 107.6)
- added Q2: IRF540N, Package_TO_SOT_THT:TO-220-3_Vertical, F.Cu at (104.5, 196.6)
- added R1: 10k, Resistor_THT:R_Axial_DIN0204_L3.6mm_D1.6mm_P7.62mm_Horizontal, F.Cu at (110.5, 148.1)
- added R1: 10k, Resistor_THT:R_Axial_DIN0204_L3.6mm_D1.6mm_P7.62mm_Horizontal, F.Cu at (110.5, 237.1)
- added R10: 10k, Resistor_THT:R_Axial_DIN0204_L3.6mm_D1.6mm_P7.62mm_Horizontal, F.Cu at (61.8, 152.1)
- added R10: 10k, Resistor_THT:R_Axial_DIN0204_L3.6mm_D1.6mm_P7.62mm_Horizontal, F.Cu at (61.8, 241.1)
- added R11: 1k, Resistor_THT:R_Axial_DIN0204_L3.6mm_D1.6mm_P7.62mm_Horizontal, F.Cu at (107.0, 143.2)
- added R11: 1k, Resistor_THT:R_Axial_DIN0204_L3.6mm_D1.6mm_P7.62mm_Horizontal, F.Cu at (107.0, 232.2)
- added R12: 100k, Resistor_THT:R_Axial_DIN0204_L3.6mm_D1.6mm_P7.62mm_Horizontal, F.Cu at (70.6, 244.6)
- added R12: 100k, Resistor_THT:R_Axial_DIN0204_L3.6mm_D1.6mm_P7.62mm_Horizontal, F.Cu at (70.6, 155.6)
- added R13: 100k, Resistor_THT:R_Axial_DIN0204_L3.6mm_D1.6mm_P7.62mm_Horizontal, F.Cu at (70.8, 166.3)
- added R13: 100k, Resistor_THT:R_Axial_DIN0204_L3.6mm_D1.6mm_P7.62mm_Horizontal, F.Cu at (70.8, 255.3)
- added R14: 5k6, Resistor_THT:R_Axial_DIN0204_L3.6mm_D1.6mm_P7.62mm_Horizontal, F.Cu at (128.9, 176.2)
- added R14: 5k6, Resistor_THT:R_Axial_DIN0204_L3.6mm_D1.6mm_P7.62mm_Horizontal, F.Cu at (128.9, 265.2)
- added R15: 33k, Resistor_THT:R_Axial_DIN0204_L3.6mm_D1.6mm_P7.62mm_Horizontal, F.Cu at (107.7, 176.2)
- added R15: 33k, Resistor_THT:R_Axial_DIN0204_L3.6mm_D1.6mm_P7.62mm_Horizontal, F.Cu at (107.7, 265.2)
- added R16: 100k, Resistor_THT:R_Axial_DIN0204_L3.6mm_D1.6mm_P7.62mm_Horizontal, F.Cu at (118.4, 265.2)
- added R16: 100k, Resistor_THT:R_Axial_DIN0204_L3.6mm_D1.6mm_P7.62mm_Horizontal, F.Cu at (118.4, 176.2)
- added R17: 1k, Resistor_THT:R_Axial_DIN0204_L3.6mm_D1.6mm_P7.62mm_Horizontal, F.Cu at (139.4, 176.2)
- added R17: 1k, Resistor_THT:R_Axial_DIN0204_L3.6mm_D1.6mm_P7.62mm_Horizontal, F.Cu at (139.4, 265.2)
- added R2: 30k, Resistor_THT:R_Axial_DIN0204_L3.6mm_D1.6mm_P7.62mm_Horizontal, F.Cu at (99.1, 148.2)
- added R2: 30k, Resistor_THT:R_Axial_DIN0204_L3.6mm_D1.6mm_P7.62mm_Horizontal, F.Cu at (99.1, 237.2)
- added R3: 33k, Resistor_THT:R_Axial_DIN0204_L3.6mm_D1.6mm_P7.62mm_Horizontal, F.Cu at (132.6, 148.1)
- added R3: 33k, Resistor_THT:R_Axial_DIN0204_L3.6mm_D1.6mm_P7.62mm_Horizontal, F.Cu at (132.6, 237.1)
- added R4: 56k, Resistor_THT:R_Axial_DIN0204_L3.6mm_D1.6mm_P7.62mm_Horizontal, F.Cu at (140.9, 144.6)
- added R4: 56k, Resistor_THT:R_Axial_DIN0204_L3.6mm_D1.6mm_P7.62mm_Horizontal, F.Cu at (140.9, 233.6)
- added R5: 10k, Resistor_THT:R_Axial_DIN0204_L3.6mm_D1.6mm_P7.62mm_Horizontal, F.Cu at (145.9, 156.0)
- added R5: 10k, Resistor_THT:R_Axial_DIN0204_L3.6mm_D1.6mm_P7.62mm_Horizontal, F.Cu at (145.9, 245.0)
- added R6: 56k, Resistor_THT:R_Axial_DIN0204_L3.6mm_D1.6mm_P7.62mm_Horizontal, F.Cu at (145.9, 233.5)
- added R6: 56k, Resistor_THT:R_Axial_DIN0204_L3.6mm_D1.6mm_P7.62mm_Horizontal, F.Cu at (146.5, 59.4)
- added R6: 56k, Resistor_THT:R_Axial_DIN0204_L3.6mm_D1.6mm_P7.62mm_Horizontal, F.Cu at (145.9, 144.5)
- added R7: ~, Resistor_THT:R_Axial_DIN0204_L3.6mm_D1.6mm_P7.62mm_Horizontal, F.Cu at (138.2, 113.6)
- added R7: ~, Resistor_THT:R_Axial_DIN0204_L3.6mm_D1.6mm_P7.62mm_Horizontal, F.Cu at (138.9, 28.5)
- added R7: ~, Resistor_THT:R_Axial_DIN0204_L3.6mm_D1.6mm_P7.62mm_Horizontal, F.Cu at (138.2, 202.6)
- added R8: 1k, Resistor_THT:R_Axial_DIN0204_L3.6mm_D1.6mm_P7.62mm_Horizontal, F.Cu at (61.8, 164.6)
- added R8: 1k, Resistor_THT:R_Axial_DIN0204_L3.6mm_D1.6mm_P7.62mm_Horizontal, F.Cu at (61.8, 253.6)
- added R9: 10k, Resistor_THT:R_Axial_DIN0204_L3.6mm_D1.6mm_P7.62mm_Horizontal, F.Cu at (61.8, 247.1)
- added R9: 10k, Resistor_THT:R_Axial_DIN0204_L3.6mm_D1.6mm_P7.62mm_Horizontal, F.Cu at (61.8, 158.1)
- added REF**: MountingHole_3.2mm_M3, MountingHole:MountingHole_3.2mm_M3, F.Cu at (146.9, 193.4)
- added REF**: MountingHole_3.2mm_M3, MountingHole:MountingHole_3.2mm_M3, F.Cu at (146.9, 104.4)
- added REF**: MountingHole_3.2mm_M3, MountingHole:MountingHole_3.2mm_M3, F.Cu at (147.5, 19.2)
- added TL1: TL431LP, Package_TO_SOT_THT:TO-92_HandSolder, F.Cu at (56.8, 261.5)
- added TL1: TL431LP, Package_TO_SOT_THT:TO-92_HandSolder, F.Cu at (56.8, 172.5)
- added U1: TL082, Package_DIP:DIP-8_W7.62mm_Socket, F.Cu at (102.2, 244.3)
- added U1: TL082, Package_DIP:DIP-8_W7.62mm_Socket, F.Cu at (102.2, 155.3)
- added U1: TL082, Package_DIP:DIP-8_W7.62mm_Socket, F.Cu at (102.9, 70.2)
- added U2: IR2111, Package_DIP:DIP-8_W7.62mm_Socket, F.Cu at (79.6, 249.6)
- added U2: IR2111, Package_DIP:DIP-8_W7.62mm_Socket, F.Cu at (79.6, 160.6)
- added U2: IR2111, Package_DIP:DIP-8_W7.62mm_Socket, F.Cu at (80.2, 75.5)
- added VEE1: VEE, Connector_PinHeader_2.00mm:PinHeader_1x01_P2.00mm_Vertical, F.Cu at (54.5, 228.1)
- added VEE1: VEE, Connector_PinHeader_2.00mm:PinHeader_1x01_P2.00mm_Vertical, F.Cu at (54.5, 139.1)
- added Vctrl_H1: Vctrl_H, Connector_PinHeader_2.00mm:PinHeader_1x01_P2.00mm_Vertical, F.Cu at (81.0, 226.1)
- added Vctrl_H1: Vctrl_H, Connector_PinHeader_2.00mm:PinHeader_1x01_P2.00mm_Vertical, F.Cu at (81.0, 137.1)
- added Vctrl_L1: Vctrl_L, Connector_PinHeader_2.00mm:PinHeader_1x01_P2.00mm_Vertical, F.Cu at (89.3, 226.1)
- added Vctrl_L1: Vctrl_L, Connector_PinHeader_2.00mm:PinHeader_1x01_P2.00mm_Vertical, F.Cu at (89.3, 137.1)
- added Vo1: Vo, Connector_PinHeader_2.00mm:PinHeader_1x01_P2.00mm_Vertical, F.Cu at (142.7, 139.4)
- added Vo1: Vo, Connector_PinHeader_2.00mm:PinHeader_1x01_P2.00mm_Vertical, F.Cu at (142.7, 228.4)
- BC1: renamed from BC546; value BC546 -> ~
- R10: renamed from R5; value 1k -> 10k
- R17: renamed from R13; value 100 -> 1k
- R3: renamed from R9; value 22k -> 33k
- R4: renamed from R1; value 10k -> 56k
- R9: renamed from R4; value 1k -> 10k
- moved R5 3.47 mm to (146.5, 70.9)
- moved R4 1.91 mm to (141.5, 59.5)
- renumbered C6 to C2, C2 to C3, C5 to C4, C4 to C5, C3 to C6, MBR735 to D2, J2 to J4, Q3 to Q1, Q4 to Q2, R10 to R1, R14 to R11, R11 to R12, R12 to R13, R8 to R14, R6 to R15, R7 to R16, R15 to R2, R2 to R5, R3 to R8, TL431 to TL1
Connections:
- C6 pad 2: /VEE -> /Vs
- D1 pad 2: /Vo -> Net-(D1-A)
- L1 pad 1: Net-(Q3-S) -> /Vs
- Q1 pad 3: Net-(Q3-S) -> /Vs
- Q2 pad 2: Net-(Q3-S) -> /Vs
- R4 pad 2: /v_muestra -> Net-(J3-Pin_1)
- R5 pad 1: /v_muestra -> Net-(J3-Pin_1)
Routing:
- net Net-(J5-Pin_1): track 0.00 -> 428.4 mm
- net GND: track 313.7 -> 603.9 mm, vias 0 -> 12
- net /Vs: track 0.00 -> 255.3 mm, vias 0 -> 6
- net Net-(LM1B-+): track 67.7 -> 294.9 mm
- net /PWM: track 344.0 -> 148.8 mm, vias 0 -> 6
- net /VEE: track 451.2 -> 624.7 mm, vias 0 -> 6
- net /V_cuad: track 33.8 -> 173.0 mm
- net /Vcc5: track 262.6 -> 388.5 mm, vias 0 -> 18
- net /V_triag: track 55.2 -> 179.1 mm
- net Net-(U1A--): track 103.0 -> 202.3 mm
- net /Vmed: track 186.0 -> 260.8 mm, vias 0 -> 24
- net /Vctrl_H: track 167.4 -> 240.6 mm, vias 0 -> 6
- net Net-(Q3-S): track 68.7 -> 0.00 mm
- net /v_muestra: track 106.7 -> 170.1 mm, vias 0 -> 6
- net /Vo: track 227.3 -> 285.0 mm
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Other:
- board size 100.3 x 249.4 mm -> 100.6 x 254.1 mm
